File: LEDBoard_1x4_16bit_highdensity.sch (KiCad schematic (older format))
At the start: 10 parts, among them J1 signal_in, J2 signal_out, J3 power, U1 TLC5971PWP

Commit message: partly routed
Connections:
- net labels added: IREF
Changed lines of the file:
@@
 F 3 "~" H 3750 4500 50  0001 C CNN
 	1    3750 4500
-	1    0    0    -1
+	-1   0    0    -1
 $EndComp
 $Comp
@@
 	7550 5350 7550 5150
 Connection ~ 7550 5150
+Text Label 3750 3550 0    50   ~ 0
+IREF
 $EndSCHEMATC
