File: LEDBoard_1x4_16bit_highdensity.sch (KiCad schematic (older format))
At the start: 10 parts, among them J1 signal_in, J2 signal_out, J3 power, U1 TLC5971PWP

Commit message: basic component placement done
Parts:
- D1, D2, D3, D4: footprint LED_SMD:LED_Avago_PLCC6_3x2.8mm -> LEDs_SMD_NICHIA:LED_NSSM124_PCBEdge
- J1, J2, J3: footprint Connector_PinHeader_1.27mm:PinHeader_1x02_P1.27mm_Vertical -> Resistor_SMD:R_0402_1005Metric
- U1: footprint Package_SO:HTSSOP-20-1EP_4.4x6.5mm_P0.65mm_EP3.4x6.5mm_ThermalVias -> Package_DFN_QFN:VQFN-24-1EP_4x4mm_P0.5mm_EP2.45x2.45mm_ThermalVias; symbol Driver_LED_mod:TLC5971PWP -> Driver_LED_mod:TLC5971RGET
Changed lines of the file:
@@
 $EndDescr
 $Comp
-L Driver_LED_mod:TLC5971PWP U1
+L Driver_LED_mod:TLC5971RGET U1
 U 1 1 5B6971A6
 P 4650 3850
 F 0 "U1" H 4150 4850 50  0000 C CNN
 F 1 "TLC5971PWP" H 5000 4850 50  0000 C CNN
-F 2 "Package_SO:HTSSOP-20-1EP_4.4x6.5mm_P0.65mm_EP3.4x6.5mm_ThermalVias" H 4100 5000 50  0001 L CNN
+F 2 "Package_DFN_QFN:VQFN-24-1EP_4x4mm_P0.5mm_EP2.45x2.45mm_ThermalVias" H 4100 5000 50  0001 L CNN
 F 3 "http://www.ti.com/lit/ds/symlink/tlc5971.pdf" H 4650 3550 50  0001 C CNN
 	1    4650 3850
@@
 F 0 "J3" H 5330 6292 50  0000 L CNN
 F 1 "power" H 5330 6201 50  0000 L CNN
-F 2 "Connector_PinHeader_1.27mm:PinHeader_1x02_P1.27mm_Vertical" H 5250 6300 50  0001 C CNN
+F 2 "Resistor_SMD:R_0402_1005Metric" H 5250 6300 50  0001 C CNN
 F 3 "~" H 5250 6300 50  0001 C CNN
 	1    5250 6300
@@
 F 0 "J1" H 3220 3025 50  0000 C CNN
 F 1 "signal_in" H 3220 3116 50  0000 C CNN
-F 2 "Connector_PinHeader_1.27mm:PinHeader_1x02_P1.27mm_Vertical" H 3300 3350 50  0001 C CNN
+F 2 "Resistor_SMD:R_0402_1005Metric" H 3300 3350 50  0001 C CNN
 F 3 "~" H 3300 3350 50  0001 C CNN
 	1    3300 3350
@@
 F 0 "J2" H 6080 3242 50  0000 L CNN
 F 1 "signal_out" H 6080 3151 50  0000 L CNN
-F 2 "Connector_PinHeader_1.27mm:PinHeader_1x02_P1.27mm_Vertical" H 6000 3250 50  0001 C CNN
+F 2 "Resistor_SMD:R_0402_1005Metric" H 6000 3250 50  0001 C CNN
 F 3 "~" H 6000 3250 50  0001 C CNN
 	1    6000 3250
@@
 F 0 "D1" H 7150 2897 50  0000 C CNN
 F 1 "led_0" H 7150 2806 50  0000 C CNN
-F 2 "LED_SMD:LED_Avago_PLCC6_3x2.8mm" H 7150 2350 50  0001 C CNN
+F 2 "LEDs_SMD_NICHIA:LED_NSSM124_PCBEdge" H 7150 2350 50  0001 C CNN
 F 3 "~" H 7150 2350 50  0001 C CNN
 	1    7150 2400
@@
 F 0 "D2" H 7150 3797 50  0000 C CNN
 F 1 "led_1" H 7150 3706 50  0000 C CNN
-F 2 "LED_SMD:LED_Avago_PLCC6_3x2.8mm" H 7150 3250 50  0001 C CNN
+F 2 "LEDs_SMD_NICHIA:LED_NSSM124_PCBEdge" H 7150 3250 50  0001 C CNN
 F 3 "~" H 7150 3250 50  0001 C CNN
 	1    7150 3300
@@
 F 0 "D3" H 7150 4747 50  0000 C CNN
 F 1 "led_2" H 7150 4656 50  0000 C CNN
-F 2 "LED_SMD:LED_Avago_PLCC6_3x2.8mm" H 7150 4200 50  0001 C CNN
+F 2 "LEDs_SMD_NICHIA:LED_NSSM124_PCBEdge" H 7150 4200 50  0001 C CNN
 F 3 "~" H 7150 4200 50  0001 C CNN
 	1    7150 4250
@@
 F 0 "D4" H 7150 5647 50  0000 C CNN
 F 1 "led_3" H 7150 5556 50  0000 C CNN
-F 2 "LED_SMD:LED_Avago_PLCC6_3x2.8mm" H 7150 5100 50  0001 C CNN
+F 2 "LEDs_SMD_NICHIA:LED_NSSM124_PCBEdge" H 7150 5100 50  0001 C CNN
 F 3 "~" H 7150 5100 50  0001 C CNN
 	1    7150 5150

Commit message: placing & layout done :-)
Parts:
- U1: footprint Package_DFN_QFN:VQFN-24-1EP_4x4mm_P0.5mm_EP2.45x2.45mm_ThermalVias -> Package_SO:HTSSOP-20-1EP_4.4x6.5mm_P0.65mm_EP3.4x6.5mm_ThermalVias; symbol Driver_LED_mod:TLC5971RGET -> Driver_LED_mod:TLC5971PWP
Changed lines of the file:
@@
 $EndDescr
 $Comp
-L Driver_LED_mod:TLC5971RGET U1
+L Driver_LED_mod:TLC5971PWP U1
 U 1 1 5B6971A6
 P 4650 3850
-F 0 "U1" H 4150 4850 50  0000 C CNN
-F 1 "TLC5971PWP" H 5000 4850 50  0000 C CNN
-F 2 "Package_DFN_QFN:VQFN-24-1EP_4x4mm_P0.5mm_EP2.45x2.45mm_ThermalVias" H 4100 5000 50  0001 L CNN
+F 0 "U1" H 4100 4850 50  0000 L CNN
+F 1 "TLC5971PWP" H 4700 4850 50  0000 L CNN
+F 2 "Package_SO:HTSSOP-20-1EP_4.4x6.5mm_P0.65mm_EP3.4x6.5mm_ThermalVias" H 4100 5000 50  0001 L CNN
 F 3 "http://www.ti.com/lit/ds/symlink/tlc5971.pdf" H 4650 3550 50  0001 C CNN
 	1    4650 3850

Commit message: first placement test
Parts:
- D1, D2, D3, D4: footprint LEDs_SMD_NICHIA:LED_NSSM124_PCBEdge -> LEDs_SMD_NICHIA:LED_NSSM124_wViaHeatSinkBig_roundedPads
- U1: footprint Package_SO:HTSSOP-20-1EP_4.4x6.5mm_P0.65mm_EP3.4x6.5mm_ThermalVias -> Package_SO_mod:HTSSOP-20-1EP_4.4x6.5mm_P0.65mm_EP3.4x6.5mm_Mask2.75x3.43mm_ThermalVias_HandSolder
Changed lines of the file:
@@
 F 0 "U1" H 4100 4850 50  0000 L CNN
 F 1 "TLC5971PWP" H 4700 4850 50  0000 L CNN
-F 2 "Package_SO:HTSSOP-20-1EP_4.4x6.5mm_P0.65mm_EP3.4x6.5mm_ThermalVias" H 4100 5000 50  0001 L CNN
+F 2 "Package_SO_mod:HTSSOP-20-1EP_4.4x6.5mm_P0.65mm_EP3.4x6.5mm_Mask2.75x3.43mm_ThermalVias_HandSolder" H 4100 5000 50  0001 L CNN
 F 3 "http://www.ti.com/lit/ds/symlink/tlc5971.pdf" H 4650 3550 50  0001 C CNN
 	1    4650 3850
@@
 F 0 "D1" H 7150 2897 50  0000 C CNN
 F 1 "led_0" H 7150 2806 50  0000 C CNN
-F 2 "LEDs_SMD_NICHIA:LED_NSSM124_PCBEdge" H 7150 2350 50  0001 C CNN
+F 2 "LEDs_SMD_NICHIA:LED_NSSM124_wViaHeatSinkBig_roundedPads" H 7150 2350 50  0001 C CNN
 F 3 "~" H 7150 2350 50  0001 C CNN
 	1    7150 2400
@@
 F 0 "D2" H 7150 3797 50  0000 C CNN
 F 1 "led_1" H 7150 3706 50  0000 C CNN
-F 2 "LEDs_SMD_NICHIA:LED_NSSM124_PCBEdge" H 7150 3250 50  0001 C CNN
+F 2 "LEDs_SMD_NICHIA:LED_NSSM124_wViaHeatSinkBig_roundedPads" H 7150 3250 50  0001 C CNN
 F 3 "~" H 7150 3250 50  0001 C CNN
 	1    7150 3300
@@
 F 0 "D3" H 7150 4747 50  0000 C CNN
 F 1 "led_2" H 7150 4656 50  0000 C CNN
-F 2 "LEDs_SMD_NICHIA:LED_NSSM124_PCBEdge" H 7150 4200 50  0001 C CNN
+F 2 "LEDs_SMD_NICHIA:LED_NSSM124_wViaHeatSinkBig_roundedPads" H 7150 4200 50  0001 C CNN
 F 3 "~" H 7150 4200 50  0001 C CNN
 	1    7150 4250
@@
 F 0 "D4" H 7150 5647 50  0000 C CNN
 F 1 "led_3" H 7150 5556 50  0000 C CNN
-F 2 "LEDs_SMD_NICHIA:LED_NSSM124_PCBEdge" H 7150 5100 50  0001 C CNN
+F 2 "LEDs_SMD_NICHIA:LED_NSSM124_wViaHeatSinkBig_roundedPads" H 7150 5100 50  0001 C CNN
 F 3 "~" H 7150 5100 50  0001 C CNN
 	1    7150 5150

Commit message: prepared amulet version
Parts:
- D1, D2, D3, D4: footprint LEDs_SMD_NICHIA:LED_NSSM124_wViaHeatSinkBig_roundedPads -> LEDs_SMD_NICHIA:LED_NSSM124
- U1: footprint Package_SO_mod:HTSSOP-20-1EP_4.4x6.5mm_P0.65mm_EP3.4x6.5mm_Mask2.75x3.43mm_ThermalVias_HandSolder -> Package_DFN_QFN:Texas_RGE0024H_EP2.7x2.7mm_ThermalVias; symbol Driver_LED_mod:TLC5971PWP -> Driver_LED:TLC5971RGE
Connections:
- wire segments 29 -> 28
Changed lines of the file:
@@
 $EndDescr
 $Comp
-L Driver_LED_mod:TLC5971PWP U1
+L Driver_LED:TLC5971RGE U1
 U 1 1 5B6971A6
 P 4650 3850
-F 0 "U1" H 4100 4850 50  0000 L CNN
-F 1 "TLC5971PWP" H 4700 4850 50  0000 L CNN
-F 2 "Package_SO_mod:HTSSOP-20-1EP_4.4x6.5mm_P0.65mm_EP3.4x6.5mm_Mask2.75x3.43mm_ThermalVias_HandSolder" H 4100 5000 50  0001 L CNN
-F 3 "http://www.ti.com/lit/ds/symlink/tlc5971.pdf" H 4650 3550 50  0001 C CNN
+F 0 "U1" H 4700 4600 50  0000 L CNN
+F 1 "TLC5971PWP" H 4700 3100 50  0000 L CNN
+F 2 "Package_DFN_QFN:Texas_RGE0024H_EP2.7x2.7mm_ThermalVias" H 4700 3000 50  0001 L CNN
+F 3 "" H 4650 3550 50  0001 C CNN
 	1    4650 3850
 	1    0    0    -1
@@
 L Connector_Generic:Conn_01x02 J3
 U 1 1 5B697371
-P 5250 6300
-F 0 "J3" H 5330 6292 50  0000 L CNN
-F 1 "power" H 5330 6201 50  0000 L CNN
-F 2 "Resistor_SMD:R_0402_1005Metric" H 5250 6300 50  0001 C CNN
-F 3 "~" H 5250 6300 50  0001 C CNN
-	1    5250 6300
+P 5500 5200
+F 0 "J3" H 5580 5192 50  0000 L CNN
+F 1 "power" H 5580 5101 50  0000 L CNN
+F 2 "Resistor_SMD:R_0402_1005Metric" H 5500 5200 50  0001 C CNN
+F 3 "~" H 5500 5200 50  0001 C CNN
+	1    5500 5200
 	-1   0    0    1
 $EndComp
@@
 L Connector_Generic:Conn_01x02 J1
 U 1 1 5B697555
-P 3300 3350
-F 0 "J1" H 3220 3025 50  0000 C CNN
-F 1 "signal_in" H 3220 3116 50  0000 C CNN
-F 2 "Resistor_SMD:R_0402_1005Metric" H 3300 3350 50  0001 C CNN
-F 3 "~" H 3300 3350 50  0001 C CNN
-	1    3300 3350
+P 3500 3750
+F 0 "J1" H 3600 3650 50  0000 C CNN
+F 1 "signal_in" H 3750 3750 50  0000 C CNN
+F 2 "Resistor_SMD:R_0402_1005Metric" H 3500 3750 50  0001 C CNN
+F 3 "~" H 3500 3750 50  0001 C CNN
+	1    3500 3750
 	-1   0    0    1
 $EndComp
@@
 L Connector_Generic:Conn_01x02 J2
 U 1 1 5B69763E
-P 6000 3250
-F 0 "J2" H 6080 3242 50  0000 L CNN
-F 1 "signal_out" H 6080 3151 50  0000 L CNN
-F 2 "Resistor_SMD:R_0402_1005Metric" H 6000 3250 50  0001 C CNN
-F 3 "~" H 6000 3250 50  0001 C CNN
-	1    6000 3250
-	1    0    0    -1
-$EndComp
-Wire Wire Line
-	3500 3250 3950 3250
-Wire Wire Line
-	3950 3350 3500 3350
-Wire Wire Line
-	5350 3250 5800 3250
-Wire Wire Line
-	5350 3350 5800 3350
-Text Label 3550 3250 0    50   ~ 0
+P 3500 3950
+F 0 "J2" H 3580 3942 50  0000 L CNN
+F 1 "signal_out" H 3580 3851 50  0000 L CNN
+F 2 "Resistor_SMD:R_0402_1005Metric" H 3500 3950 50  0001 C CNN
+F 3 "~" H 3500 3950 50  0001 C CNN
+	1    3500 3950
+	-1   0    0    -1
+$EndComp
+Wire Wire Line
+	3700 3650 4150 3650
+Wire Wire Line
+	4150 3750 3700 3750
+Wire Wire Line
+	4150 3950 3700 3950
+Wire Wire Line
+	4150 4050 3700 4050
+Text Label 4150 3650 2    50   ~ 0
 clock_in
-Text Label 3550 3350 0    50   ~ 0
+Text Label 4150 3750 2    50   ~ 0
 data_in
-Text Label 5400 3250 0    50   ~ 0
+Text Label 4150 3950 2    50   ~ 0
 clock_out
-Text Label 5400 3350 0    50   ~ 0
+Text Label 4150 4050 2    50   ~ 0
 data_out
-$Comp
-L power:GND #PWR0101
-U 1 1 5B69A47A
-P 4550 4950
-F 0 "#PWR0101" H 4550 4700 50  0001 C CNN
-F 1 "GND" H 4555 4777 50  0000 C CNN
-F 2 "" H 4550 4950 50  0001 C CNN
-F 3 "" H 4550 4950 50  0001 C CNN
-	1    4550 4950
-	1    0    0    -1
-$EndComp
 $Comp
 L power:GND #PWR0102
 U 1 1 5B69A4AC
-P 4750 4950
-F 0 "#PWR0102" H 4750 4700 50  0001 C CNN
-F 1 "GND" H 4755 4777 50  0000 C CNN
-F 2 "" H 4750 4950 50  0001 C CNN
-F 3 "" H 4750 4950 50  0001 C CNN
-	1    4750 4950
+P 4650 4650
+F 0 "#PWR0102" H 4650 4400 50  0001 C CNN
+F 1 "GND" H 4655 4477 50  0000 C CNN
+F 2 "" H 4650 4650 50  0001 C CNN
+F 3 "" H 4650 4650 50  0001 C CNN
+	1    4650 4650
 	1    0    0    -1
 $EndComp
@@
 L power:GND #PWR0103
 U 1 1 5B69A55A
-P 5450 6300
-F 0 "#PWR0103" H 5450 6050 50  0001 C CNN
-F 1 "GND" H 5455 6127 50  0000 C CNN
-F 2 "" H 5450 6300 50  0001 C CNN
-F 3 "" H 5450 6300 50  0001 C CNN
-	1    5450 6300
+P 5700 5200
+F 0 "#PWR0103" H 5700 4950 50  0001 C CNN
+F 1 "GND" H 5705 5027 50  0000 C CNN
+F 2 "" H 5700 5200 50  0001 C CNN
+F 3 "" H 5700 5200 50  0001 C CNN
+	1    5700 5200
 	1    0    0    -1
 $EndComp
@@
 L power:VCC #PWR0104
 U 1 1 5B69A64F
-P 5450 6200
-F 0 "#PWR0104" H 5450 6050 50  0001 C CNN
-F 1 "VCC" H 5467 6373 50  0000 C CNN
-F 2 "" H 5450 6200 50  0001 C CNN
-F 3 "" H 5450 6200 50  0001 C CNN
-	1    5450 6200
+P 5700 5100
+F 0 "#PWR0104" H 5700 4950 50  0001 C CNN
+F 1 "VCC" H 5717 5273 50  0000 C CNN
+F 2 "" H 5700 5100 50  0001 C CNN
+F 3 "" H 5700 5100 50  0001 C CNN
+	1    5700 5100
 	1    0    0    -1
 $EndComp
@@
 L power:VCC #PWR0105
 U 1 1 5B69A669
-P 4650 2750
-F 0 "#PWR0105" H 4650 2600 50  0001 C CNN
-F 1 "VCC" H 4667 2923 50  0000 C CNN
-F 2 "" H 4650 2750 50  0001 C CNN
-F 3 "" H 4650 2750 50  0001 C CNN
-	1    4650 2750
+P 4450 3050
+F 0 "#PWR0105" H 4450 2900 50  0001 C CNN
+F 1 "VCC" H 4467 3223 50  0000 C CNN
+F 2 "" H 4450 3050 50  0001 C CNN
+F 3 "" H 4450 3050 50  0001 C CNN
+	1    4450 3050
 	1    0    0    -1
 $EndComp
@@
 L power:VCC #PWR0106
 U 1 1 5B69A74C
-P 3750 4400
-F 0 "#PWR0106" H 3750 4250 50  0001 C CNN
-F 1 "VCC" H 3767 4573 50  0000 C CNN
-F 2 "" H 3750 4400 50  0001 C CNN
-F 3 "" H 3750 4400 50  0001 C CNN
-	1    3750 4400
+P 4000 3100
+F 0 "#PWR0106" H 4000 2950 50  0001 C CNN
+F 1 "VCC" H 4017 3273 50  0000 C CNN
+F 2 "" H 4000 3100 50  0001 C CNN
+F 3 "" H 4000 3100 50  0001 C CNN
+	1    4000 3100
 	1    0    0    -1
 $EndComp
@@
 L power:GND #PWR0107
 U 1 1 5B69A763
-P 3750 4600
-F 0 "#PWR0107" H 3750 4350 50  0001 C CNN
-F 1 "GND" H 3755 4427 50  0000 C CNN
-F 2 "" H 3750 4600 50  0001 C CNN
-F 3 "" H 3750 4600 50  0001 C CNN
-	1    3750 4600
+P 4000 3300
+F 0 "#PWR0107" H 4000 3050 50  0001 C CNN
+F 1 "GND" H 4005 3127 50  0000 C CNN
+F 2 "" H 4000 3300 50  0001 C CNN
+F 3 "" H 4000 3300 50  0001 C CNN
+	1    4000 3300
 	1    0    0    -1
 $EndComp
@@
 L Device:C_Small C1
 U 1 1 5B69A7A7
-P 3750 4500
-F 0 "C1" H 3842 4546 50  0000 L CNN
-F 1 "100n" H 3842 4455 50  0000 L CNN
-F 2 "Capacitor_SMD:C_0603_1608Metric_Pad1.05x0.95mm_HandSolder" H 3750 4500 50  0001 C CNN
-F 3 "~" H 3750 4500 50  0001 C CNN
-	1    3750 4500
-	1    0    0    -1
+P 4000 3200
+F 0 "C1" H 4092 3246 50  0000 L CNN
+F 1 "100n" H 4092 3155 50  0000 L CNN
+F 2 "Capacitor_SMD:C_0603_1608Metric_Pad1.05x0.95mm_HandSolder" H 4000 3200 50  0001 C CNN
+F 3 "~" H 4000 3200 50  0001 C CNN
+	1    4000 3200
+	-1   0    0    -1
 $EndComp
 $Comp
 L Device:R R1
 U 1 1 5B69AAAA
-P 3750 3700
-F 0 "R1" H 3820 3746 50  0000 L CNN
-F 1 "2k7" H 3820 3655 50  0000 L CNN
-F 2 "Resistor_SMD:R_0603_1608Metric_Pad1.05x0.95mm_HandSolder" V 3680 3700 50  0001 C CNN
-F 3 "~" H 3750 3700 50  0001 C CNN
-	1    3750 3700
-	1    0    0    -1
-$EndComp
-Wire Wire Line
-	3750 3550 3950 3550
+P 4450 4800
+F 0 "R1" H 4520 4846 50  0000 L CNN
+F 1 "2k7" H 4520 4755 50  0000 L CNN
+F 2 "Resistor_SMD:R_0603_1608Metric_Pad1.05x0.95mm_HandSolder" V 4380 4800 50  0001 C CNN
+F 3 "~" H 4450 4800 50  0001 C CNN
+	1    4450 4800
+	-1   0    0    -1
+$EndComp
 $Comp
 L power:GND #PWR0108
 U 1 1 5B69AB7A
-P 3750 3850
-F 0 "#PWR0108" H 3750 3600 50  0001 C CNN
-F 1 "GND" H 3755 3677 50  0000 C CNN
-F 2 "" H 3750 3850 50  0001 C CNN
-F 3 "" H 3750 3850 50  0001 C CNN
-	1    3750 3850
+P 4450 4950
+F 0 "#PWR0108" H 4450 4700 50  0001 C CNN
+F 1 "GND" H 4455 4777 50  0000 C CNN
+F 2 "" H 4450 4950 50  0001 C CNN
+F 3 "" H 4450 4950 50  0001 C CNN
+	1    4450 4950
 	1    0    0    -1
 $EndComp
@@
 L power:VCC #PWR0109
 U 1 1 5B69AC72
-P 5350 3050
-F 0 "#PWR0109" H 5350 2900 50  0001 C CNN
-F 1 "VCC" H 5367 3223 50  0000 C CNN
-F 2 "" H 5350 3050 50  0001 C CNN
-F 3 "" H 5350 3050 50  0001 C CNN
-	1    5350 3050
-	1    0    0    -1
-$EndComp
-Text Label 5350 3550 0    50   ~ 0
+P 4650 3050
+F 0 "#PWR0109" H 4650 2900 50  0001 C CNN
+F 1 "VCC" H 4667 3223 50  0000 C CNN
+F 2 "" H 4650 3050 50  0001 C CNN
+F 3 "" H 4650 3050 50  0001 C CNN
+	1    4650 3050
+	1    0    0    -1
+$EndComp
+Text Label 5150 3250 0    50   ~ 0
 led_0_r
-Text Label 5350 3850 0    50   ~ 0
+Text Label 5150 3550 0    50   ~ 0
 led_1_r
-Text Label 5350 4150 0    50   ~ 0
+Text Label 5150 3850 0    50   ~ 0
 led_2_r
-Text Label 5350 4450 0    50   ~ 0
+Text Label 5150 4150 0    50   ~ 0
 led_3_r
-Text Label 5350 3650 0    50   ~ 0
+Text Label 5150 3350 0    50   ~ 0
 led_0_g
-Text Label 5350 3950 0    50   ~ 0
+Text Label 5150 3650 0    50   ~ 0
 led_1_g
-Text Label 5350 4250 0    50   ~ 0
+Text Label 5150 3950 0    50   ~ 0
 led_2_g
-Text Label 5350 4550 0    50   ~ 0
+Text Label 5150 4250 0    50   ~ 0
 led_3_g
-Text Label 5350 3750 0    50   ~ 0
+Text Label 5150 3450 0    50   ~ 0
 led_0_b
-Text Label 5350 4050 0    50   ~ 0
+Text Label 5150 3750 0    50   ~ 0
 led_1_b
-Text Label 5350 4350 0    50   ~ 0
+Text Label 5150 4050 0    50   ~ 0
 led_2_b
-Text Label 5350 4650 0    50   ~ 0
+Text Label 5150 4350 0    50   ~ 0
 led_3_b
 Text Label 6950 2200 2    50   ~ 0
@@
 F 0 "D1" H 7150 2897 50  0000 C CNN
 F 1 "led_0" H 7150 2806 50  0000 C CNN
-F 2 "LEDs_SMD_NICHIA:LED_NSSM124_wViaHeatSinkBig_roundedPads" H 7150 2350 50  0001 C CNN
+F 2 "LEDs_SMD_NICHIA:LED_NSSM124" H 7150 2350 50  0001 C CNN
 F 3 "~" H 7150 2350 50  0001 C CNN
 	1    7150 2400
@@
 F 0 "D2" H 7150 3797 50  0000 C CNN
 F 1 "led_1" H 7150 3706 50  0000 C CNN
-F 2 "LEDs_SMD_NICHIA:LED_NSSM124_wViaHeatSinkBig_roundedPads" H 7150 3250 50  0001 C CNN
+F 2 "LEDs_SMD_NICHIA:LED_NSSM124" H 7150 3250 50  0001 C CNN
 F 3 "~" H 7150 3250 50  0001 C CNN
 	1    7150 3300
@@
 F 0 "D3" H 7150 4747 50  0000 C CNN
 F 1 "led_2" H 7150 4656 50  0000 C CNN
-F 2 "LEDs_SMD_NICHIA:LED_NSSM124_wViaHeatSinkBig_roundedPads" H 7150 4200 50  0001 C CNN
+F 2 "LEDs_SMD_NICHIA:LED_NSSM124" H 7150 4200 50  0001 C CNN
 F 3 "~" H 7150 4200 50  0001 C CNN
 	1    7150 4250
@@
 F 0 "D4" H 7150 5647 50  0000 C CNN
 F 1 "led_3" H 7150 5556 50  0000 C CNN
-F 2 "LEDs_SMD_NICHIA:LED_NSSM124_wViaHeatSinkBig_roundedPads" H 7150 5100 50  0001 C CNN
+F 2 "LEDs_SMD_NICHIA:LED_NSSM124" H 7150 5100 50  0001 C CNN
 F 3 "~" H 7150 5100 50  0001 C CNN
 	1    7150 5150
